File: EAGLE/Projects/EPS Flatsat Module/EPS Flatsat Module/EPS Flatsat Module.sch (EAGLE design)
At the start: 2 parts, among them J1 ESQ-126-39-G-D, J2 ESQ-126-39-G-D

Commit message: Updates to flatsat module. Added MSP430 headers, DCDC converters, and some power switches to schematic. Did some placement on the board layout.
Parts:
- added C1, C2: (no value), rcl:C-USC0805
- added C10, C5, C6, C7, C8, C9: 1u, rcl:C-USC0805
- added C3, C4: (no value), rcl:CPOL-USE2.5-6
- added D1, D2: 1N4004, diode:1N4004
- added J3, J4: TSW-110-23-F-D, TSW-110-23-F-D:TSW-110-23-F-D
- added PS1: R-543.3PA, R-543.3PA:R-543.3PA
- added PS2: R-545.0PA, R-545.0PA:R-545.0PA
- added R1, R2, R3, R4, R5, R6: 10k, rcl:R-US_R0805
- added T1, T2: 2N3904, transistor:2N3904
- added U1, U2, U3, U4, U5, U6: Value, TPS27081ADDCR:TPS27081ADDCR
Connections:
- new net 3V3ONOFF: T1.B
- new net 3V3SYS: C10.1, C3.+, C8.1, C9.1, D1.A, J2.27, J2.28, PS1.VOUT, PS1.VOUT(AUTO_SENSE), R4.1, R5.1, R6.1, U4.VIN, U5.VIN, U6.VIN
- new net 5VONOFF: T2.B
- new net 5VSYS: C4.+, C5.1, C6.1, C7.1, D2.A, J2.25, J2.26, PS2.VOUT, PS2.VOUT(AUTO_SENSE), R1.1, R2.1, R3.1, U1.VIN, U2.VIN, U3.VIN
- new net GND: C1.2, C10.2, C2.2, C3.-, C4.-, C5.2, C6.2, C7.2, C8.2, C9.2, J2.14, J2.17, J2.21, J2.22, J2.29, J2.30, J2.32, J2.47, J2.48, J2.9, J3.04, J4.02, PS1.GND, PS2.GND, T1.E, T2.E, U1.R2, U2.R2, U3.R2, U4.R2, U5.R2, U6.R2
- new net N$1: PS1.!ON/OFF, T1.C
- new net N$2: PS2.!ON/OFF, T2.C
- new net N$3: R1.2, U1.R1_C1
- new net N$4: R2.2, U2.R1_C1
- new net N$5: R3.2, U3.R1_C1
- new net N$6: R4.2, U4.R1_C1
- new net N$7: R5.2, U5.R1_C1
- new net N$8: R6.2, U6.R1_C1
- new net PDM10: J2.20, U6.VOUT, U6.VOUT_2
- new net PDM10EN: U6.ON_OFF
- new net PDM5: J2.13, U1.VOUT, U1.VOUT_2
- new net PDM5EN: U1.ON_OFF
- new net PDM6: J2.15, U2.VOUT, U2.VOUT_2
- new net PDM6EN: U2.ON_OFF
- new net PDM7: J2.16, U3.VOUT, U3.VOUT_2
- new net PDM7EN: U3.ON_OFF
- new net PDM8: J2.18, U4.VOUT, U4.VOUT_2
- new net PDM8EN: U4.ON_OFF
- new net PDM9: J2.19, U5.VOUT, U5.VOUT_2
- new net PDM9EN: U5.ON_OFF
- new net SCL: J1.43, J4.14
- new net SDA: J1.41, J4.12
- new net VIN: C1.1, C2.1, D1.C, D2.C, PS1.VIN, PS2.VIN
