File: EAGLE/Projects/EPS Flatsat Module/EPS Flatsat Module/EPS Flatsat Module2.sch (EAGLE design)
At the start: 51 parts, among them J1 ESQ-126-39-G-D, J2 ESQ-126-39-G-D, J5 1985881, T1 2N3904, T2 2N3904, U1 Value, U2 Value, U3 Value, U4 Value, U5 Value, U6 Value

Commit message: Added current sensing
Parts:
- removed JP2, JP3: -, Arduino-connectors:PINHD-1X15-CASTELLATED
- added C11, C12, C13, C14, C15, C16: 0.1u, rcl:C-USC0805
- added C17, C18, C19, C20, C21, C22: 0.1uF, rcl:C-USC0805
- added LED9: (no value), led:LEDCHIP-LED0805
- added R15: (no value), rcl:R-US_R0805
- added R16, R17, R18, R19, R20, R21: 0.01, rcl:R-US_R2512
- added U$1: NANO, Arduino-clone:NANO
- added U10, U11, U12, U7, U8, U9: ADM4073HWRJZ-REEL7, ADM4073HWRJZ-REEL7:ADM4073HWRJZ-REEL7
Connections:
- removed net N$19: J2.51
- removed net PDM10: J2.20, LED8.A, U6.VOUT, U6.VOUT_2
- removed net PDM10EN: JP3.8, U6.ON_OFF
- removed net PDM7: J2.16, LED6.A, U3.VOUT, U3.VOUT_2
- removed net PDM7EN: JP3.11, U3.ON_OFF
- removed net PDM8: J2.18, LED4.A, U4.VOUT, U4.VOUT_2
- removed net PDM8EN: JP3.10, U4.ON_OFF
- removed net PDM9: J2.19, LED7.A, U5.VOUT, U5.VOUT_2
- removed net PDM9EN: JP3.9, U5.ON_OFF
- new net ADC0: U$1.A3, U11.OUT
- new net ADC1: U$1.A2, U7.OUT
- new net ADC2: U$1.A1, U9.OUT
- new net ADC3: U$1.A0, U8.OUT
- new net ADC4: U$1.A6, U12.OUT
- new net ADC5: U$1.A7, U10.OUT
- new net N$18: LED9.A, U$1.D13
- new net N$27: LED9.C, R15.2
- new net PDM1: C15.1, C18.1, LED4.A, R17.1, U4.VOUT, U4.VOUT_2, U7.RS+, U7.VCC
- new net PDM1EN: U$1.D7, U4.ON_OFF
- new net PDM1_OUT: J2.17, R17.2, U7.RS-
- new net PDM2: C11.1, C17.1, LED8.A, R16.1, U6.VOUT, U6.VOUT_2, U8.RS+, U8.VCC
- new net PDM2EN: U$1.D5, U6.ON_OFF
- new net PDM2_OUT: J2.19, R16.2, U8.RS-
- new net PDM3: C16.1, C19.1, LED7.A, R18.1, U5.VOUT, U5.VOUT_2, U9.RS+, U9.VCC
- new net PDM3EN: U$1.D6, U5.ON_OFF
- new net PDM3_OUT: J2.20, R18.2, U9.RS-
- new net PDM4: C14.1, C20.1, LED6.A, R19.1, U10.RS+, U10.VCC, U3.VOUT, U3.VOUT_2
- new net PDM4EN: U$1.D8, U3.ON_OFF
- new net PDM4_OUT: J2.15, R19.2, U10.RS-
- new net PDM5_OUT: J2.16, R20.2, U11.RS-
- new net PDM6_OUT: J2.14, R21.2, U12.RS-
- net 3V3ONOFF: now also U$1.D12; no longer JP3.15
- net 5VONOFF: now also U$1.D11; no longer JP3.14
- net GND: now also C11.2, C12.2, C13.2, C14.2, C15.2, C16.2, C17.2, C18.2, C19.2, C20.2, C21.2, C22.2, J2.10, J2.13, J2.18, J2.31, J2.51, R15.1, U$1.GND, U10.GND, U10.GND_2, U11.GND, U11.GND_2, U12.GND, U12.GND_2, U7.GND, U7.GND_2, U8.GND, U8.GND_2, U9.GND, U9.GND_2; no longer J2.14, J2.17, J2.32, J2.9, JP2.14
- net PDM5: now also C13.1, C21.1, LED5.A, R20.1, U11.RS+, U11.VCC, U2.VOUT, U2.VOUT_2; no longer J2.13, LED3.A, U1.VOUT, U1.VOUT_2
- net PDM5EN: now also U$1.D9, U2.ON_OFF; no longer JP3.13, U1.ON_OFF
- net PDM6: now also C12.1, C22.1, LED3.A, R21.1, U1.VOUT, U1.VOUT_2, U12.RS+, U12.VCC; no longer J2.15, LED5.A, U2.VOUT, U2.VOUT_2
- net PDM6EN: now also U$1.D10, U1.ON_OFF; no longer JP3.12, U2.ON_OFF
- net SCL: now also J1.44, U$1.A5; no longer J1.43, JP2.9
- net SDA: now also J1.42, U$1.A4; no longer J1.41, JP2.8
- net VIN: now also U$1.RAW; no longer JP2.15
